File: AS3320.sch (KiCad schematic (older format))
At the start: 27 parts, among them J1 AudioJack2, J2 AudioJack2, J3 AudioJack2, U3 AS3320

Commit message: Refactor
Parts:
- removed C6: C, symbol Device:C
- added C5: 1µF, Capacitor_THT:CP_Radial_D5.0mm_P2.50mm, symbol Device:C_Polarized
- added J3, J4: Conn_01x01_Male, Connector_Pin:Pin_D1.0mm_L10.0mm, symbol Connector:Conn_01x01_Male
- C1: renamed from C2; footprint (none) -> Capacitor_THT:CP_Radial_D5.0mm_P2.50mm
- C2: renamed from C3; footprint (none) -> Capacitor_THT:CP_Radial_D5.0mm_P2.50mm
- C3: renamed from C4; footprint (none) -> Capacitor_THT:CP_Radial_D5.0mm_P2.50mm
- C4: renamed from C5; footprint (none) -> Capacitor_THT:CP_Radial_D5.0mm_P2.50mm
- J1, J2: footprint (none) -> Connector_AudioJacks:Jack_6.35mm_Neutrik_NJ2FD-V_Vertical
- J5: renamed from J3; footprint (none) -> Connector_AudioJacks:Jack_6.35mm_Neutrik_NJ2FD-V_Vertical
- R10: renamed from R19; footprint (none) -> Resistor_THT:R_Axial_DIN0207_L6.3mm_D2.5mm_P10.16mm_Horizontal
- R11: renamed from R20; footprint (none) -> Resistor_THT:R_Axial_DIN0207_L6.3mm_D2.5mm_P10.16mm_Horizontal
- R12: renamed from R21; footprint (none) -> Resistor_THT:R_Axial_DIN0207_L6.3mm_D2.5mm_P10.16mm_Horizontal
- R13: renamed from R22; footprint (none) -> Resistor_THT:R_Axial_DIN0207_L6.3mm_D2.5mm_P10.16mm_Horizontal
- R14: renamed from R23; footprint (none) -> Resistor_THT:R_Axial_DIN0207_L6.3mm_D2.5mm_P10.16mm_Horizontal
- R15: renamed from R24; footprint (none) -> Resistor_THT:R_Axial_DIN0207_L6.3mm_D2.5mm_P10.16mm_Horizontal
- R16: renamed from R25; footprint (none) -> Resistor_THT:R_Axial_DIN0207_L6.3mm_D2.5mm_P10.16mm_Horizontal
- R17: renamed from R26; footprint (none) -> Resistor_THT:R_Axial_DIN0207_L6.3mm_D2.5mm_P10.16mm_Horizontal
- R18: renamed from R27; footprint (none) -> Resistor_THT:R_Axial_DIN0207_L6.3mm_D2.5mm_P10.16mm_Horizontal
- R19: renamed from R28; footprint (none) -> Resistor_THT:R_Axial_DIN0207_L6.3mm_D2.5mm_P10.16mm_Horizontal
- R4: renamed from R17; footprint (none) -> Resistor_THT:R_Axial_DIN0207_L6.3mm_D2.5mm_P10.16mm_Horizontal
- R5: renamed from R16; footprint (none) -> Resistor_THT:R_Axial_DIN0207_L6.3mm_D2.5mm_P10.16mm_Horizontal
- R6: renamed from R13; footprint (none) -> Resistor_THT:R_Axial_DIN0207_L6.3mm_D2.5mm_P10.16mm_Horizontal
- R7: renamed from R14; footprint (none) -> Resistor_THT:R_Axial_DIN0207_L6.3mm_D2.5mm_P10.16mm_Horizontal
- R8: renamed from R15; footprint (none) -> Resistor_THT:R_Axial_DIN0207_L6.3mm_D2.5mm_P10.16mm_Horizontal
- R9: renamed from R18; footprint (none) -> Resistor_THT:R_Axial_DIN0207_L6.3mm_D2.5mm_P10.16mm_Horizontal
- RV7: renamed from RV8; footprint (none) -> Potentiometer_THT:Potentiometer_ACP_CA9-V10_Vertical
- RV8: renamed from RV7; footprint (none) -> Potentiometer_THT:Potentiometer_ACP_CA9-V10_Vertical
- renumbered U3 to U2
Connections:
- net labels added: +12V, -12V
- net labels removed: +15V, -15V
- wire segments 81 -> 77
Other:
- moved on the sheet: C1, C2, C3, C4, J1, J2, J5, R10, R11, R12, R13, R14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
