File: VCO-0.kicad_pcb (KiCad board)
At the start: 2 copper layers, 13 parts, among them SW1 SW_Push, SW2 SW_Push, U1 RC1602A

Commit message: Refactor
Parts:
- added C1: 300pF, Capacitor_THT:CP_Radial_D5.0mm_P2.50mm, F.Cu at (292.1, -377.2)
- added C2: 300pF, Capacitor_THT:CP_Radial_D5.0mm_P2.50mm, F.Cu at (292.1, -388.6)
- added C3: 300pF, Capacitor_THT:CP_Radial_D5.0mm_P2.50mm, F.Cu at (292.1, -364.5)
- added C4: 300pF, Capacitor_THT:CP_Radial_D5.0mm_P2.50mm, F.Cu at (292.1, -353.1)
- added C5: 1µF, Capacitor_THT:CP_Radial_D5.0mm_P2.50mm, F.Cu at (292.1, -341.6)
- added J1: AudioJack2, Connector_AudioJacks:Jack_6.35mm_Neutrik_NJ2FD-V_Vertical, F.Cu at (208.3, -334.0)
- added J2: AudioJack2, Connector_AudioJacks:Jack_6.35mm_Neutrik_NJ2FD-V_Vertical, F.Cu at (208.3, -304.8)
- added J3: Conn_01x01_Male, Connector_Pin:Pin_D1.0mm_L10.0mm, F.Cu at (309.9, -306.1)
- added J4: Conn_01x01_Male, Connector_Pin:Pin_D1.0mm_L10.0mm, F.Cu at (309.9, -322.6)
- added J5: AudioJack2, Connector_AudioJacks:Jack_6.35mm_Neutrik_NJ2FD-V_Vertical, F.Cu at (208.3, -278.1)
- added R10: 91K, Resistor_THT:R_Axial_DIN0207_L6.3mm_D2.5mm_P10.16mm_Horizontal, F.Cu at (269.1, -314.5)
- added R11: 100K, Resistor_THT:R_Axial_DIN0207_L6.3mm_D2.5mm_P10.16mm_Horizontal, F.Cu at (278.1, -304.8)
- added R12: 91K, Resistor_THT:R_Axial_DIN0207_L6.3mm_D2.5mm_P10.16mm_Horizontal, F.Cu at (247.7, -315.0)
- added R13: 100K, Resistor_THT:R_Axial_DIN0207_L6.3mm_D2.5mm_P10.16mm_Horizontal, F.Cu at (226.1, -292.1)
- added R14: 91K, Resistor_THT:R_Axial_DIN0207_L6.3mm_D2.5mm_P10.16mm_Horizontal, F.Cu at (226.1, -281.9)
- added R15: 100K, Resistor_THT:R_Axial_DIN0207_L6.3mm_D2.5mm_P10.16mm_Horizontal, F.Cu at (247.7, -281.9)
- added R16: 91K, Resistor_THT:R_Axial_DIN0207_L6.3mm_D2.5mm_P10.16mm_Horizontal, F.Cu at (248.9, -303.5)
- added R17: 100K, Resistor_THT:R_Axial_DIN0207_L6.3mm_D2.5mm_P10.16mm_Horizontal, F.Cu at (226.1, -271.8)
- added R18: 1K8, Resistor_THT:R_Axial_DIN0207_L6.3mm_D2.5mm_P10.16mm_Horizontal, F.Cu at (247.7, -271.8)
- added R19: 51K, Resistor_THT:R_Axial_DIN0207_L6.3mm_D2.5mm_P10.16mm_Horizontal, F.Cu at (226.1, -303.5)
- added R4: 100K, Resistor_THT:R_Axial_DIN0207_L6.3mm_D2.5mm_P10.16mm_Horizontal, F.Cu at (270.5, -285.8)
- added R5: 100K, Resistor_THT:R_Axial_DIN0207_L6.3mm_D2.5mm_P10.16mm_Horizontal, F.Cu at (226.1, -313.7)
- added R6: 220K, Resistor_THT:R_Axial_DIN0207_L6.3mm_D2.5mm_P10.16mm_Horizontal, F.Cu at (236.2, -387.4)
- added R7: 220K, Resistor_THT:R_Axial_DIN0207_L6.3mm_D2.5mm_P10.16mm_Horizontal, F.Cu at (247.7, -293.4)
- added R8: 220K, Resistor_THT:R_Axial_DIN0207_L6.3mm_D2.5mm_P10.16mm_Horizontal, F.Cu at (236.2, -396.2)
- added R9: 1K8, Resistor_THT:R_Axial_DIN0207_L6.3mm_D2.5mm_P10.16mm_Horizontal, F.Cu at (236.2, -379.7)
- added RV6: R_Potentiometer_Trim, Potentiometer_THT:Potentiometer_ACP_CA9-V10_Vertical, F.Cu at (-20.3, -294.6)
- added RV7: 100K, Potentiometer_THT:Potentiometer_ACP_CA9-V10_Vertical, F.Cu at (203.2, -349.2)
- added RV8: 100K, Potentiometer_THT:Potentiometer_ACP_CA9-V10_Vertical, F.Cu at (203.2, -369.6)
- added U2: AS3320, Package_DIP:DIP-18_W7.62mm, F.Cu at (240.0, -353.1)
- R1: value 330R -> 10K
- R3: value 10K -> 330R
- moved RV2 20.8 mm to (44.5, -388.6)
- moved RV1 7.62 mm to (86.4, -383.5)
- moved RV5 5.08 mm to (134.6, -381.0)
Connections:
- R1 pad 2: Net-(D1-Pad1) -> Net-(R1-Pad2)
- R2 pad 2: Net-(R1-Pad1) -> Net-(R1-Pad2)
- R3 pad 1: Net-(R3-Pad1) -> Net-(R1-Pad2)
- R3 pad 2: Net-(R1-Pad1) -> Net-(D1-Pad1)
- RV1 pad 3: Net-(R1-Pad1) -> Net-(R1-Pad2)
- RV2 pad 3: Net-(R1-Pad1) -> Net-(R1-Pad2)
- RV3 pad 3: Net-(R1-Pad1) -> Net-(R1-Pad2)
- RV4 pad 3: Net-(R1-Pad1) -> Net-(R1-Pad2)
- RV5 pad 3: Net-(R1-Pad1) -> Net-(R1-Pad2)
- SW1 pad 1: Net-(R2-Pad1) -> Net-(R1-Pad1)
- SW2 pad 1: Net-(R3-Pad1) -> Net-(R2-Pad1)
- U1 pad 1: Net-(R1-Pad1) -> Net-(R1-Pad2)
- U1 pad 16: Net-(R1-Pad1) -> Net-(R1-Pad2)
- U1 pad 5: Net-(R1-Pad1) -> Net-(R1-Pad2)
- XA1 pad D10: Net-(XA1-PadD10) -> Net-(U1-Pad14)
- XA1 pad D11: Net-(U1-Pad12) -> Net-(XA1-PadD11)
- XA1 pad D12: Net-(U1-Pad13) -> Net-(XA1-PadD12)
- XA1 pad D13: Net-(U1-Pad14) -> Net-(XA1-PadD13)
- XA1 pad D24: Net-(R2-Pad1) -> Net-(R1-Pad1)
- XA1 pad D26: Net-(R3-Pad1) -> Net-(R2-Pad1)
- XA1 pad D7: Net-(XA1-PadD7) -> Net-(U1-Pad11)
- XA1 pad D8: Net-(U1-Pad11) -> Net-(U1-Pad12)
- XA1 pad D9: Net-(XA1-PadD9) -> Net-(U1-Pad13)
- XA1 pad GND1: Net-(R1-Pad1) -> Net-(R1-Pad2)
Routing:
- net Net-(R1-Pad2): track 0.00 -> 314.8 mm, vias 0 -> 3
- net GND: track 0.00 -> 268.7 mm
- net Net-(R4-Pad1): track 0.00 -> 157.0 mm, vias 0 -> 2
- net Net-(R16-Pad1): track 0.00 -> 155.0 mm
- net Net-(D1-Pad1): track 11.4 -> 162.8 mm, vias 0 -> 1
- net Net-(R12-Pad1): track 0.00 -> 137.4 mm
- net -12V: track 0.00 -> 132.1 mm
- net Net-(R1-Pad1): track 266.1 -> 371.2 mm, vias 0 -> 3
- net Net-(R14-Pad1): track 0.00 -> 93.0 mm
- net Net-(C5-Pad2): track 0.00 -> 85.3 mm
- net Net-(R10-Pad1): track 0.00 -> 79.4 mm, vias 0 -> 1
- net Net-(J4-Pad1): track 0.00 -> 77.3 mm
- net Net-(C2-Pad1): track 0.00 -> 76.2 mm, vias 0 -> 1
- net Net-(R5-Pad1): track 0.00 -> 75.4 mm
- net +12V: track 0.00 -> 72.0 mm
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